Commit message: successful swing ; optimizing to imitate human movement ; swing then balance (to enhance)

File: ur5_robot_best.urdf (robot description, URDF)
Before this commit: robot ur5, 12 links, 11 joints
Links:
- link pendulum_link: mass 0.005 -> 0.001
Joints:
- joint pendulum_joint: limit lower=-0.4 upper=0.4 effort=0 velocity=1 -> lower=-6.28318530718 upper=6.28318530718
