Commit message: Clean repo with working balancing notebook and urdf_file

File: ur5_robot_working_balancing.urdf (robot description, URDF)
Before this commit: robot ur5, 11 links, 10 joints
Links:
- removed link tool0
- added link pendulum_link, mass 0.001; collision cylinder length=0.25 radius=0.0025; visual cylinder length=0.25 radius=0.0025
- added link pendulum_mass, mass 0.05; collision sphere radius=0.03; visual sphere radius=0.03
Joints:
- removed joint wrist_3_link-tool0_fixed_joint
- added joint pendulum_joint: type revolute, parent ee_link, child pendulum_link, origin xyz=0 0 0 rpy=0 3.1416 0, axis 0 0 1, limit lower=-6.28318530718 upper=6.28318530718
- added joint pendulum_mass_joint: type fixed, parent pendulum_link, child pendulum_mass, origin xyz=0 0 -0.25 rpy=0 0 0
- joint wrist_2_joint: limit lower=-6.28318530718 upper=6.28318530718 effort=28.0 velocity=3.2 -> lower=-0.223598776  upper=0.223598776  effort=28.0 velocity=1.2

Commit message: Better robot model + physics  and balancing

File: ur5_robot_working_balancing.urdf (robot description, URDF)
Before this commit: robot ur5, 12 links, 11 joints
Links:
- link pendulum_link: mass 0.001 -> 0.01
Joints:
- joint pendulum_joint: axis 0 0 1 -> 1 0 0; limit lower=-6.28318530718 upper=6.28318530718 -> lower=-66.28318530718 upper=66.28318530718
- joint wrist_2_joint: limit lower=-0.223598776  upper=0.223598776  effort=28.0 velocity=1.2 -> lower=-0.063598776  upper=0.063598776  effort=28.0 velocity=1.2
- joint wrist_3_joint: axis 0 1 0 -> (none); limit lower=-6.28318530718 upper=6.28318530718 effort=28.0 velocity=3.2 -> (none); origin xyz=0.0 0.0 0.09465 rpy=0.0 0.0 0.0 -> xyz=0.0 0.0 0.09465 rpy=0.0 -2.98 0.0; type revolute -> fixed
